Commit message: macro added

File: ros2_ws/src/robot_description/urdf/base/koubot_base.xacro (robot description, xacro)
@@ -9,4 +9,7 @@
     <xacro:property name="wheel_radius" value="0.04"/>
     <xacro:property name="wheel_length" value="0.036"/>
+    <xacro:property name="base_link_to_wheel_x" value="0.05"/>
+    <xacro:property name="base_link_to_wheel_y" value="0.114"/>
+    <xacro:property name="base_link_to_wheel_z" value="0.04"/>
     <xacro:property name="pi_value" value="3.141592654"/>
     <xacro:property name="half_pi" value="1.570796327"/>
@@ -76,5 +79,5 @@
     <!-- Joint - base_link / front left wheel -->
     <joint name="joint_base_link_front_left_wheel" type="continuous">
-        <origin rpy="0 0 0" xyz="0.05 0.114 -0.04" />
+        <origin rpy="0 0 0" xyz="${base_link_to_wheel_x} ${base_link_to_wheel_y} -${base_link_to_wheel_z}" />
         <child link="front_left_wheel" />
         <parent link="base_link" />
@@ -105,5 +108,5 @@
     <!-- Joint - base_link / front right wheel -->
     <joint name="joint_base_link_front_right_wheel" type="continuous">
-        <origin rpy="0 0 0" xyz="0.05 -0.114 -0.04" />
+        <origin rpy="0 0 0" xyz="${base_link_to_wheel_x} -${base_link_to_wheel_y} -${base_link_to_wheel_z}" />
         <child link="front_right_wheel" />
         <parent link="base_link" />
@@ -134,5 +137,5 @@
     <!-- Joint - base_link / back right wheel -->
     <joint name="joint_base_link_back_right_wheel" type="continuous">
-        <origin rpy="0 0 0" xyz="-0.05 -0.114 -0.04" />
+        <origin rpy="0 0 0" xyz="-${base_link_to_wheel_x} -${base_link_to_wheel_y} -${base_link_to_wheel_z}" />
         <child link="back_right_wheel" />
         <parent link="base_link" />
@@ -163,5 +166,5 @@
     <!-- Joint - base_link / back left wheel -->
     <joint name="joint_base_link_back_left_wheel" type="continuous">
-        <origin rpy="0 0 0" xyz="-0.05 0.114 -0.04" />
+        <origin rpy="0 0 0" xyz="-${base_link_to_wheel_x} ${base_link_to_wheel_y} -${base_link_to_wheel_z}" />
         <child link="back_left_wheel" />
         <parent link="base_link" />

Commit message: URDF: corrected collisions and inertias

File: ros2_ws/src/robot_description/urdf/base/koubot_base.xacro (robot description, xacro)
@@ -9,36 +9,38 @@
     <xacro:property name="wheel_radius" value="0.04"/>
     <xacro:property name="wheel_length" value="0.036"/>
-    <xacro:property name="base_link_to_wheel_x" value="0.05"/>
-    <xacro:property name="base_link_to_wheel_y" value="0.114"/>
-    <xacro:property name="base_link_to_wheel_z" value="0.04"/>
-    <xacro:property name="pi_value" value="3.141592654"/>
-    <xacro:property name="half_pi" value="1.570796327"/>
-    <!--%%%%%%%%%%%%%%%%%%%%%%%%%%%%%%%%%%%%%%%%%%%%%%%%%%%%%%%%%%%%%%%%%%%%%%%%%%%%%%%%%%%%%%%%%%%%%%%%%%%%%-->
-    <!--This will make the SDF conversion to keep links binded with FIXED JOINTS separate.-->
-    <!-- <gazebo reference="base_link_front_caster_wheel">
-        <preserveFixedJoint>true</preserveFixedJoint>
-    </gazebo>
-    <gazebo reference="base_link_back_caster_wheel">
-        <preserveFixedJoint>true</preserveFixedJoint>
-    </gazebo> -->
-    <!-- <gazebo reference="front_laser_joint">
-        <preserveFixedJoint>true</preserveFixedJoint>
-    </gazebo> -->
-    <!--Friction added here-->
+    <xacro:property name="wheel_offset_x" value="0.05"/>
+    <xacro:property name="wheel_offset_y" value="0.114"/>
+    <xacro:property name="wheel_offset_z" value="0.04"/>
+    <xacro:property name="M_PI" value="3.141592654"/>
+    <!--%%%%%%%%%%%%%%%%%%%%%%%%%%%%%%%%%%%%%%%%%%% FRICTION & STIFNESS %%%%%%%%%%%%%%%%%%%%%%%%%%%%%%%%%%%%%%%%%%%%%%%%%%%%%%%%-->
+    <!--
+    mu1: The static friction coefficient. It is how much friction there is until the object starts moving in simple terms.
+    mu2: The dynamic friction coefficient. It is how much friction there is when the object moves in simple terms.
+    kp: This coefficient sets the static contact stiffness. This determines whether the linked material is closer to marble (rigid, bigger values) or more like rubber (soft material, lower values).
+    kd: This coefficient sets the dynamic contact stiffness. This determines whether the linked material is closer to marble (rigid, bigger values) or more like rubber (soft material, lower values). It is essentially how much it deforms over a long period, exerting its pressure.
+    -->
     <gazebo reference="front_left_wheel">
-        <mu1>1</mu1>
-        <mu2>1</mu2>
+        <!-- <kp>1000000000000000000000000000.0</kp>
+        <kd>1000000000000000000000000000.0</kd> -->
+        <mu1>0.1</mu1>
+        <mu2>0.1</mu2>
     </gazebo>
     <gazebo reference="front_right_wheel">
-        <mu1>1</mu1>
-        <mu2>1</mu2>
+        <!-- <kp>1000000000000000000000000000.0</kp>
+        <kd>1000000000000000000000000000.0</kd> -->
+        <mu1>0.1</mu1>
+        <mu2>0.1</mu2>
     </gazebo>
     <gazebo reference="back_left_wheel">
-        <mu1>1</mu1>
-        <mu2>1</mu2>
+        <!-- <kp>1000000000000000000000000000.0</kp>
+        <kd>1000000000000000000000000000.0</kd> -->
+        <mu1>0.1</mu1>
+        <mu2>0.1</mu2>
     </gazebo>
     <gazebo reference="back_right_wheel">
-        <mu1>1</mu1>
-        <mu2>1</mu2>
+        <!-- <kp>1000000000000000000000000000.0</kp>
+        <kd>1000000000000000000000000000.0</kd> -->
+        <mu1>0.1</mu1>
+        <mu2>0.1</mu2>
     </gazebo>
     <!--%%%%%%%%%%%%%%%%%%%%%%%%%%%%%%%%%%%%%%%%%%%%%%%%%%%%%%%%%%%%%%%%%%%%%%%%%%%%%%%%%%%%%%%%%%%%%%%%%%%%%-->
@@ -65,5 +67,5 @@
         </inertial>
         <collision>
-            <origin xyz="0 0 0" rpy="0 0 0" />
+            <origin xyz="0 0 0" rpy="0 0 ${M_PI/2}" />
             <geometry>
                 <box size="${chassis_width} ${chassis_depth} ${chassis_height}" />
@@ -71,5 +73,5 @@
         </collision>
         <visual>
-            <origin xyz="0 0 -${chassis_height/2}" rpy="-${half_pi} 0 0" />
+            <origin xyz="0 0 -${chassis_height/2}" rpy="-${M_PI/2} 0 0" />
             <geometry>
                 <mesh filename="package://robot_description/meshes/chassis.dae"/>
@@ -79,5 +81,5 @@
     <!-- Joint - base_link / front left wheel -->
     <joint name="joint_base_link_front_left_wheel" type="continuous">
-        <origin rpy="0 0 0" xyz="${base_link_to_wheel_x} ${base_link_to_wheel_y} -${base_link_to_wheel_z}" />
+        <origin rpy="0 0 0" xyz="${wheel_offset_x} ${wheel_offset_y} -${wheel_offset_z}" />
         <child link="front_left_wheel" />
         <parent link="base_link" />
@@ -90,15 +92,15 @@
         <inertial>
             <mass value="${wheel_mass}" />
-            <origin xyz="0 0 0" rpy="0 0 0" />
-            <inertia ixx="0.000254" ixy="0" ixz="0" iyy="0.000254" iyz="0" izz="0.0004"/>
-        </inertial>
-        <collision>
-            <origin rpy="${pi_value} 0 0" xyz="0 0 0" />
-            <geometry>
-                <cylinder length="${wheel_length}" radius="${wheel_radius}"/>
-            </geometry>
-        </collision>
-        <visual>
-            <origin rpy="${pi_value} 0 0" xyz="0 0 0" />
+            <origin xyz="0 0 0" rpy="${M_PI/2} 0 0" />
+            <inertia ixx="0.000254" ixy="0" ixz="0" iyy="0.000254" iyz="0" izz="0.0004"/>
+        </inertial>
+        <collision>
+            <origin rpy="${M_PI/2} 0 0" xyz="0 0 0" />
+            <geometry>
+                <cylinder length="${wheel_length}" radius="${wheel_radius}"/>
+            </geometry>
+        </collision>
+        <visual>
+            <origin rpy="${M_PI} 0 0" xyz="0 0 0" />
             <geometry>
                 <mesh filename="package://robot_description/meshes/wheels_scaled.dae"/>
@@ -108,5 +110,5 @@
     <!-- Joint - base_link / front right wheel -->
     <joint name="joint_base_link_front_right_wheel" type="continuous">
-        <origin rpy="0 0 0" xyz="${base_link_to_wheel_x} -${base_link_to_wheel_y} -${base_link_to_wheel_z}" />
+        <origin rpy="0 0 0" xyz="${wheel_offset_x} -${wheel_offset_y} -${wheel_offset_z}" />
         <child link="front_right_wheel" />
         <parent link="base_link" />
@@ -119,15 +121,15 @@
         <inertial>
             <mass value="${wheel_mass}" />
-            <origin xyz="0 0 0" rpy="0 0 0" />
-            <inertia ixx="0.000254" ixy="0" ixz="0" iyy="0.000254" iyz="0" izz="0.0004"/>
-        </inertial>
-        <collision>
-            <origin rpy="${pi_value} 0 0" xyz="0 0 0" />
-            <geometry>
-                <cylinder length="${wheel_length}" radius="${wheel_radius}"/>
-            </geometry>
-        </collision>
-        <visual>
-            <origin rpy="${pi_value} 0 0" xyz="0 0 0" />
+            <origin xyz="0 0 0" rpy="${M_PI/2} 0 0" />
+            <inertia ixx="0.000254" ixy="0" ixz="0" iyy="0.000254" iyz="0" izz="0.0004"/>
+        </inertial>
+        <collision>
+            <origin rpy="${M_PI/2} 0 0" xyz="0 0 0" />
+            <geometry>
+                <cylinder length="${wheel_length}" radius="${wheel_radius}"/>
+            </geometry>
+        </collision>
+        <visual>
+            <origin rpy="${M_PI} 0 0" xyz="0 0 0" />
             <geometry>
                 <mesh filename="package://robot_description/meshes/wheels_scaled.dae"/>
@@ -137,5 +139,5 @@
     <!-- Joint - base_link / back right wheel -->
     <joint name="joint_base_link_back_right_wheel" type="continuous">
-        <origin rpy="0 0 0" xyz="-${base_link_to_wheel_x} -${base_link_to_wheel_y} -${base_link_to_wheel_z}" />
+        <origin rpy="0 0 0" xyz="-${wheel_offset_x} -${wheel_offset_y} -${wheel_offset_z}" />
         <child link="back_right_wheel" />
         <parent link="base_link" />
@@ -148,15 +150,15 @@
         <inertial>
             <mass value="${wheel_mass}" />
-            <origin xyz="0 0 0" rpy="0 0 0" />
-            <inertia ixx="0.000254" ixy="0" ixz="0" iyy="0.000254" iyz="0" izz="0.0004"/>
-        </inertial>
-        <collision>
-            <origin rpy="${pi_value} 0 0" xyz="0 0 0" />
-            <geometry>
-                <cylinder length="${wheel_length}" radius="${wheel_radius}"/>
-            </geometry>
-        </collision>
-        <visual>
-            <origin rpy="${pi_value} 0 0" xyz="0 0 0" />
+            <origin xyz="0 0 0" rpy="${M_PI/2} 0 0" />
+            <inertia ixx="0.000254" ixy="0" ixz="0" iyy="0.000254" iyz="0" izz="0.0004"/>
+        </inertial>
+        <collision>
+            <origin rpy="${M_PI/2} 0 0" xyz="0 0 0" />
+            <geometry>
+                <cylinder length="${wheel_length}" radius="${wheel_radius}"/>
+            </geometry>
+        </collision>
+        <visual>
+            <origin rpy="${M_PI} 0 0" xyz="0 0 0" />
             <geometry>
                 <mesh filename="package://robot_description/meshes/wheels_scaled.dae"/>
@@ -166,5 +168,5 @@
     <!-- Joint - base_link / back left wheel -->
     <joint name="joint_base_link_back_left_wheel" type="continuous">
-        <origin rpy="0 0 0" xyz="-${base_link_to_wheel_x} ${base_link_to_wheel_y} -${base_link_to_wheel_z}" />
+        <origin rpy="0 0 0" xyz="-${wheel_offset_x} ${wheel_offset_y} -${wheel_offset_z}" />
         <child link="back_left_wheel" />
         <parent link="base_link" />
@@ -177,15 +179,15 @@
         <inertial>
             <mass value="${wheel_mass}" />
-            <origin xyz="0 0 0" rpy="0 0 0" />
-            <inertia ixx="0.000254" ixy="0" ixz="0" iyy="0.000254" iyz="0" izz="0.0004"/>
-        </inertial>
-        <collision>
-            <origin rpy="${pi_value} 0 0" xyz="0 0 0" />
-            <geometry>
-                <cylinder length="${wheel_length}" radius="${wheel_radius}"/>
-            </geometry>
-        </collision>
-        <visual>
-            <origin rpy="${pi_value} 0 0" xyz="0 0 0" />
+            <origin xyz="0 0 0" rpy="${M_PI/2} 0 0" />
+            <inertia ixx="0.000254" ixy="0" ixz="0" iyy="0.000254" iyz="0" izz="0.0004"/>
+        </inertial>
+        <collision>
+            <origin rpy="${M_PI/2} 0 0" xyz="0 0 0" />
+            <geometry>
+                <cylinder length="${wheel_length}" radius="${wheel_radius}"/>
+            </geometry>
+        </collision>
+        <visual>
+            <origin rpy="${M_PI} 0 0" xyz="0 0 0" />
             <geometry>
                 <mesh filename="package://robot_description/meshes/wheels_scaled.dae"/>

Commit message: renaming wheels collada file

File: ros2_ws/src/robot_description/urdf/base/koubot_base.xacro (robot description, xacro)
@@ -104,5 +104,5 @@
             <origin rpy="${M_PI} 0 0" xyz="0 0 0" />
             <geometry>
-                <mesh filename="package://robot_description/meshes/wheels_scaled.dae"/>
+                <mesh filename="package://robot_description/meshes/wheels.dae"/>
             </geometry>
         </visual>
@@ -133,5 +133,5 @@
             <origin rpy="${M_PI} 0 0" xyz="0 0 0" />
             <geometry>
-                <mesh filename="package://robot_description/meshes/wheels_scaled.dae"/>
+                <mesh filename="package://robot_description/meshes/wheels.dae"/>
             </geometry>
         </visual>
@@ -162,5 +162,5 @@
             <origin rpy="${M_PI} 0 0" xyz="0 0 0" />
             <geometry>
-                <mesh filename="package://robot_description/meshes/wheels_scaled.dae"/>
+                <mesh filename="package://robot_description/meshes/wheels.dae"/>
             </geometry>
         </visual>
@@ -191,5 +191,5 @@
             <origin rpy="${M_PI} 0 0" xyz="0 0 0" />
             <geometry>
-                <mesh filename="package://robot_description/meshes/wheels_scaled.dae"/>
+                <mesh filename="package://robot_description/meshes/wheels.dae"/>
             </geometry>
         </visual>

Commit message: macro for inertias

File: ros2_ws/src/robot_description/urdf/base/koubot_base.xacro (robot description, xacro)
@@ -13,4 +13,11 @@
     <xacro:property name="wheel_offset_z" value="0.04"/>
     <xacro:property name="M_PI" value="3.141592654"/>
+    <!--Inertia Calculator for a Box-->
+    <xacro:macro name="box_inertia" params="mass x y z">
+        <inertia  ixx="${mass*(y*y+z*z)/12.0}" ixy = "0" ixz = "0"
+              iyy="${mass*(x*x+z*z)/12.0}" iyz = "0"
+              izz="${mass*(x*x+y*y)/12.0}"
+        />
+    </xacro:macro>
     <!--%%%%%%%%%%%%%%%%%%%%%%%%%%%%%%%%%%%%%%%%%%% FRICTION & STIFNESS %%%%%%%%%%%%%%%%%%%%%%%%%%%%%%%%%%%%%%%%%%%%%%%%%%%%%%%%-->
     <!--
@@ -64,5 +71,6 @@
             <mass value="${chassis_mass}" />
             <origin xyz="0 0 0.0" />
-            <inertia  ixx="0.015052083333333336" ixy="0.0"  ixz="0.0" iyy="0.021708333333333336"  iyz="0.0"  izz="0.02667708333333334" />
+            <xacro:box_inertia mass="${chassis_mass}" x="${chassis_depth}" y="${chassis_width}" z="${chassis_height}"/>
+            <!-- <inertia  ixx="0.015052083333333336" ixy="0.0"  ixz="0.0" iyy="0.021708333333333336"  iyz="0.0"  izz="0.02667708333333334" /> -->
         </inertial>
         <collision>

Commit message: cleaned URDF

File: ros2_ws/src/robot_description/urdf/base/koubot_base.xacro (robot description, xacro)
@@ -13,42 +13,32 @@
     <xacro:property name="wheel_offset_z" value="0.04"/>
     <xacro:property name="M_PI" value="3.141592654"/>
-    <!--Inertia Calculator for a Box-->
-    <xacro:macro name="box_inertia" params="mass x y z">
-        <inertia  ixx="${mass*(y*y+z*z)/12.0}" ixy = "0" ixz = "0"
-              iyy="${mass*(x*x+z*z)/12.0}" iyz = "0"
-              izz="${mass*(x*x+y*y)/12.0}"
+    <!--Inertia Calculator for Chassis-->
+    <xacro:macro name="chassis_inertia" params="mass_chassis x y z">
+        <inertia  ixx="${mass_chassis*(y*y+z*z)/12.0}" ixy = "0" ixz = "0"
+              iyy="${mass_chassis*(x*x+z*z)/12.0}" iyz = "0"
+              izz="${mass_chassis*(x*x+y*y)/12.0}"
+        />
+    </xacro:macro>
+    <!--Inertia Calculator for Wheels-->
+    <xacro:macro name="wheels_inertia" params="mass_wheel r h">
+        <inertia  ixx="${mass_wheel*(3*r*r + h*h)/12.0}" ixy = "0" ixz = "0"
+              iyy="${mass_wheel*(3*r*r + h*h)/12.0}" iyz = "0"
+              izz="${mass_wheel*(r*r)/2.0}"
         />
     </xacro:macro>
     <!--%%%%%%%%%%%%%%%%%%%%%%%%%%%%%%%%%%%%%%%%%%% FRICTION & STIFNESS %%%%%%%%%%%%%%%%%%%%%%%%%%%%%%%%%%%%%%%%%%%%%%%%%%%%%%%%-->
     <!--
-    mu1: The static friction coefficient. It is how much friction there is until the object starts moving in simple terms.
-    mu2: The dynamic friction coefficient. It is how much friction there is when the object moves in simple terms.
-    kp: This coefficient sets the static contact stiffness. This determines whether the linked material is closer to marble (rigid, bigger values) or more like rubber (soft material, lower values).
-    kd: This coefficient sets the dynamic contact stiffness. This determines whether the linked material is closer to marble (rigid, bigger values) or more like rubber (soft material, lower values). It is essentially how much it deforms over a long period, exerting its pressure.
+    mu1: The static friction coefficient.
+    It is how much friction there is until the object starts moving in simple terms.
+    mu2: The dynamic friction coefficient.
+    It is how much friction there is when the object moves in simple terms.
+    kp: This coefficient sets the static contact stiffness.
+    This determines whether the linked material is closer to marble (rigid, bigger values)
+    or more like rubber (soft material, lower values).
+    kd: This coefficient sets the dynamic contact stiffness.
+    This determines whether the linked material is closer to marble (rigid, bigger values)
+    or more like rubber (soft material, lower values).
+    It is essentially how much it deforms over a long period, exerting its pressure.
     -->
-    <gazebo reference="front_left_wheel">
-        <!-- <kp>1000000000000000000000000000.0</kp>
-        <kd>1000000000000000000000000000.0</kd> -->
-        <mu1>0.1</mu1>
-        <mu2>0.1</mu2>
-    </gazebo>
-    <gazebo reference="front_right_wheel">
-        <!-- <kp>1000000000000000000000000000.0</kp>
-        <kd>1000000000000000000000000000.0</kd> -->
-        <mu1>0.1</mu1>
-        <mu2>0.1</mu2>
-    </gazebo>
-    <gazebo reference="back_left_wheel">
-        <!-- <kp>1000000000000000000000000000.0</kp>
-        <kd>1000000000000000000000000000.0</kd> -->
-        <mu1>0.1</mu1>
-        <mu2>0.1</mu2>
-    </gazebo>
-    <gazebo reference="back_right_wheel">
-        <!-- <kp>1000000000000000000000000000.0</kp>
-        <kd>1000000000000000000000000000.0</kd> -->
-        <mu1>0.1</mu1>
-        <mu2>0.1</mu2>
-    </gazebo>
     <!--%%%%%%%%%%%%%%%%%%%%%%%%%%%%%%%%%%%%%%%%%%%%%%%%%%%%%%%%%%%%%%%%%%%%%%%%%%%%%%%%%%%%%%%%%%%%%%%%%%%%%-->
     <!-- BASE FOOTPRINT -->
@@ -71,6 +61,5 @@
             <mass value="${chassis_mass}" />
             <origin xyz="0 0 0.0" />
-            <xacro:box_inertia mass="${chassis_mass}" x="${chassis_depth}" y="${chassis_width}" z="${chassis_height}"/>
-            <!-- <inertia  ixx="0.015052083333333336" ixy="0.0"  ixz="0.0" iyy="0.021708333333333336"  iyz="0.0"  izz="0.02667708333333334" /> -->
+            <xacro:chassis_inertia mass_chassis="${chassis_mass}" x="${chassis_depth}" y="${chassis_width}" z="${chassis_height}"/>
         </inertial>
         <collision>
@@ -101,5 +90,5 @@
             <mass value="${wheel_mass}" />
             <origin xyz="0 0 0" rpy="${M_PI/2} 0 0" />
-            <inertia ixx="0.000254" ixy="0" ixz="0" iyy="0.000254" iyz="0" izz="0.0004"/>
+            <xacro:wheels_inertia mass_wheel="${wheel_mass}" r="${wheel_radius}" h="${wheel_length}"/>
         </inertial>
         <collision>
@@ -130,5 +119,5 @@
             <mass value="${wheel_mass}" />
             <origin xyz="0 0 0" rpy="${M_PI/2} 0 0" />
-            <inertia ixx="0.000254" ixy="0" ixz="0" iyy="0.000254" iyz="0" izz="0.0004"/>
+            <xacro:wheels_inertia mass_wheel="${wheel_mass}" r="${wheel_radius}" h="${wheel_length}"/>
         </inertial>
         <collision>
@@ -159,5 +148,5 @@
             <mass value="${wheel_mass}" />
             <origin xyz="0 0 0" rpy="${M_PI/2} 0 0" />
-            <inertia ixx="0.000254" ixy="0" ixz="0" iyy="0.000254" iyz="0" izz="0.0004"/>
+            <xacro:wheels_inertia mass_wheel="${wheel_mass}" r="${wheel_radius}" h="${wheel_length}"/>
         </inertial>
         <collision>
@@ -188,5 +177,5 @@
             <mass value="${wheel_mass}" />
             <origin xyz="0 0 0" rpy="${M_PI/2} 0 0" />
-            <inertia ixx="0.000254" ixy="0" ixz="0" iyy="0.000254" iyz="0" izz="0.0004"/>
+            <xacro:wheels_inertia mass_wheel="${wheel_mass}" r="${wheel_radius}" h="${wheel_length}"/>
         </inertial>
         <collision>
@@ -217,14 +206,4 @@
         <child link="front_laser" />
     </joint> -->
-    <!-- <xacro:include filename="$(find robot_description)/urdf/base/koubot_base.gazebo" /> -->
-    <gazebo>
-        <plugin name="omni_steering" filename="libgazebo_ros_planar_move.so">
-            <commandTopic>cmd_vel</commandTopic>
-            <odometryTopic>odom</odometryTopic>
-            <odometryFrame>odom</odometryFrame>
-            <odometryRate>20.0</odometryRate>
-            <robotBaseFrame>base_link</robotBaseFrame>
-            <publishTF>true</publishTF>  <!-- change to true ?? -->
-        </plugin>
-    </gazebo>
+    <xacro:include filename="$(find robot_description)/urdf/base/koubot_base.gazebo" />
 </robot>
